File: connectors.kicad_sch (KiCad schematic)
At the start: 5 parts, among them J2 Conn_01x04, J3 Conn_01x04, J4 Conn_01x04, J5 USB_C_Receptacle_USB2.0_16P, U3 USBLC6-4SC6

Commit message: Finished schematic and first layout
Parts:
- removed J4: Conn_01x04, symbol Connector_Generic:Conn_01x04
- removed U3: USBLC6-4SC6, Package_TO_SOT_SMD:SOT-23-6, symbol Power_Protection:USBLC6-4SC6
- added R40, R41: 0, Resistor_SMD:R_0805_2012Metric, symbol Device:R
- added R42, R43: 5.1k, Resistor_SMD:R_0805_2012Metric, symbol Device:R
- added U1: USBLC6-2SC6, Package_TO_SOT_SMD:SOT-23-6, symbol Power_Protection:USBLC6-2SC6
- J2, J3: footprint (none) -> footprints:jst_pa4
Connections:
- net GND: now reaches J2.1 (Pin_1)
- net GND: now also J3.1 (Pin_1), J5.A1 (GND), J5.A12 (GND), J5.B1 (GND), J5.B12 (GND), J5.S1 (SHIELD), R40.2, R41.2, R42.2, R43.2, U1.2 (GND)
- net +3.3V: now reaches J2.2 (Pin_2)
- net +3.3V: now also J3.2 (Pin_2)
- net sensor_1_rx: now reaches J2.3 (Pin_3)
- net sensor_1_tx: now reaches J2.4 (Pin_4)
- net sensor_2_rx: now reaches J3.3 (Pin_3)
- net sensor_2_tx: now reaches J3.4 (Pin_4)
- net +5V: now reaches J5.A4 (VBUS), J5.A9 (VBUS), J5.B4 (VBUS), J5.B9 (VBUS)
- net +5V: now also U1.5 (VBUS)
- net at J5.A5 (CC1): now also R43.1
- net at J5.A6 (D+): now also J5.B6 (D+), U1.3 (I/O2)
- net at J5.A7 (D-): now also J5.B7 (D-), U1.1 (I/O1)
- net at J5.A8 (SBU1): now also R41.1
- net at J5.B5 (CC2): now also R42.1
- net at J5.B8 (SBU2): now also R40.1
- new net usb_dm: U1.6 (I/O1)
- new net usb_dp: U1.4 (I/O2)
Other:
- note removed: "Sensor 3"
- title: (none) -> Connectors
- moved on the sheet: J2, J3, J5
