File: connectors.kicad_sch (KiCad schematic)
At the start: 8 parts, among them J2 Conn_01x04, J3 Conn_01x04, J5 USB_C_Receptacle_USB2.0_16P, U1 USBLC6-2SC6

Commit message: Updated PCB
Parts:
- renumbered J5 to J40, J2 to J41, J3 to J42, U1 to U40
Changed lines of the file:
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@@
 		(dnp no)
 		(fields_autoplaced yes)
-		(property "Reference" "J2"
+		(property "Reference" "J41"
 			(at 228.6 55.8799 0)
 			(show_name no)
@@
 			(project "weather_station"
 				(path "/934dbf27-5b13-4be9-992c-a6264d0a607d/e42933ad-d6ea-46d3-a44b-420d06a9a31d"
-					(reference "J2")
+					(reference "J41")
 					(unit 1)
 				)
@@
 		(dnp no)
 		(fields_autoplaced yes)
-		(property "Reference" "J3"
+		(property "Reference" "J42"
 			(at 228.6 106.6799 0)
 			(show_name no)
@@
 			(project "weather_station"
 				(path "/934dbf27-5b13-4be9-992c-a6264d0a607d/e42933ad-d6ea-46d3-a44b-420d06a9a31d"
-					(reference "J3")
+					(reference "J42")
 					(unit 1)
 				)
@@
 		(dnp no)
 		(fields_autoplaced yes)
-		(property "Reference" "U1"
+		(property "Reference" "U40"
 			(at 124.8411 60.96 0)
 			(show_name no)
@@
 			(project "weather_station"
 				(path "/934dbf27-5b13-4be9-992c-a6264d0a607d/e42933ad-d6ea-46d3-a44b-420d06a9a31d"
-					(reference "U1")
+					(reference "U40")
 					(unit 1)
 				)
@@
 		(dnp no)
 		(fields_autoplaced yes)
-		(property "Reference" "J5"
+		(property "Reference" "J40"
 			(at 69.85 53.34 0)
 			(show_name no)
@@
 			(project "weather_station"
 				(path "/934dbf27-5b13-4be9-992c-a6264d0a607d/e42933ad-d6ea-46d3-a44b-420d06a9a31d"
-					(reference "J5")
-					(unit 1)
-				)
+					(reference "J40")
+					(unit 1)
+				)
