File: display.kicad_sch (KiCad schematic)
At the start: 1 part, among them J1 Conn_01x10_Pin

Commit message: Finished schematic and first layout
Parts:
- added C30, C31: 0.1uF, Capacitor_SMD:C_0805_2012Metric, symbol Device:C
- added C32: 1uF, Capacitor_SMD:C_0805_2012Metric, symbol Device:C
- J1: footprint (none) -> footprints:FFC2B35-10-T
Connections:
- net display_sclk: now reaches J1.1 (Pin_1)
- net GND: now reaches J1.10 (Pin_10)
- net GND: now also J1.9 (Pin_9), C30.2, C31.2, C32.2
- net display_mosi: now reaches J1.2 (Pin_2)
- net display_cs: now reaches J1.3 (Pin_3)
- net display_extcomin: now reaches J1.4 (Pin_4)
- net +3.3V: now reaches J1.5 (Pin_5)
- net +3.3V: now also C30.1
- net +5V: now reaches J1.6 (Pin_6)
- net +5V: now also J1.7 (Pin_7), C31.1, C32.1
- net display_extmode: now reaches J1.8 (Pin_8)
Other:
- note added: "VDD"
- note added: "VDDA"
- title: (none) -> Display
- moved on the sheet: J1
