File: display.kicad_sch (KiCad schematic)
At the start: 4 parts, among them J1 Conn_01x10_Pin

Commit message: Updated PCB
Parts:
- renumbered J1 to J30
Changed lines of the file:
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@@
 		(in_pos_files yes)
 		(dnp no)
-		(property "Reference" "J1"
+		(property "Reference" "J30"
 			(at 100.965 55.88 0)
 			(show_name no)
@@
 			(project "weather_station"
 				(path "/934dbf27-5b13-4be9-992c-a6264d0a607d/18aed268-9190-456d-b983-0438bc709a2a"
-					(reference "J1")
+					(reference "J30")
 					(unit 1)
 				)

Commit message: Changed capacitor value display
Parts:
- C30, C31: value 0.1uF -> 100nF
Changed lines of the file:
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@@
 			)
 		)
-		(property "Value" "0.1uF"
+		(property "Value" "100nF"
 			(at 173.99 73.6599 0)
 			(show_name no)
@@
 			)
 		)
-		(property "Value" "0.1uF"
+		(property "Value" "100nF"
 			(at 156.21 73.6599 0)
 			(show_name no)
