File: power_supply.kicad_sch (KiCad schematic)
At the start: 1 part, among them U2 AZ1117CH2-3.3

Commit message: Finished schematic and first layout
Connections:
- net +5V: now reaches U2.1 (IN)
- net GND: now reaches U2.2 (GND)
- net +3.3V: now reaches U2.3 (OUT)
Other:
- title: (none) -> Power supply
