File: power_supply.kicad_sch (KiCad schematic)
At the start: 1 part, among them U2 AZ1117CH2-3.3

Commit message: Updated PCB
Parts:
- renumbered U2 to U10
Changed lines of the file:
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@@
 		(dnp no)
 		(fields_autoplaced yes)
-		(property "Reference" "U2"
+		(property "Reference" "U10"
 			(at 76.2 57.15 0)
 			(show_name no)
@@
 			(project "weather_station"
 				(path "/934dbf27-5b13-4be9-992c-a6264d0a607d/b80aed7d-1ea3-40c8-9a59-917a6bf113d7"
-					(reference "U2")
+					(reference "U10")
 					(unit 1)
 				)

Commit message: Updated schematic with power supply capacitors
Parts:
- added C10: 10uF, Capacitor_SMD:C_0805_2012Metric, symbol Device:C
- added C11: 22uF, Capacitor_SMD:C_0805_2012Metric, symbol Device:C
Connections:
- net +3.3V: now also C11.1
- net +5V: now also C10.1
- net GND: now also C10.2, C11.2
