File: microcontroller.kicad_sch (KiCad schematic)
At the start: 15 parts, among them J6 JTAG_connector, SW1 SW_Push, U4 STM32F103RGTx, X1 831066657

Commit message: Updated PCB
Parts:
- renumbered J6 to J20, SW1 to SW20, U4 to U20, X1 to X20
Connections:
- net diaply_cs: now also U20.24 (PC4); no longer U20.20 (PA4)
- net display_extcomin: now also U20.25 (PC5); no longer U20.24 (PC4)
- net display_extmode: now also U20.26 (PB0); no longer U20.25 (PC5)
Changed lines of the file:
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@@
 	)
 	(no_connect
-		(at 152.4 97.79)
-	)
-	(no_connect
 		(at 116.84 97.79)
 	)
@@
 	)
 	(no_connect
+		(at 152.4 64.77)
+	)
+	(no_connect
 		(at 152.4 54.61)
 	)
@@
 	(wire
 		(pts
-			(xy 152.4 64.77) (xy 157.48 64.77)
-		)
-		(stroke
-			(width 0)
-			(type default)
-		)
-	)
-	(wire
-		(pts
 			(xy 237.49 72.39) (xy 234.95 72.39)
 		)
@@
 	(wire
 		(pts
-			(xy 111.76 85.09) (xy 116.84 85.09)
-		)
-		(stroke
-			(width 0)
-			(type default)
-		)
-	)
-	(wire
-		(pts
 			(xy 33.02 41.91) (xy 33.02 48.26)
 		)
@@
 	(wire
 		(pts
+			(xy 111.76 85.09) (xy 116.84 85.09)
+		)
+		(stroke
+			(width 0)
+			(type default)
+		)
+	)
+	(wire
+		(pts
 			(xy 152.4 85.09) (xy 157.48 85.09)
 		)
@@
 	(wire
 		(pts
-			(xy 111.76 87.63) (xy 116.84 87.63)
+			(xy 152.4 72.39) (xy 157.48 72.39)
 		)
 		(stroke
@@
 	(wire
 		(pts
-			(xy 152.4 72.39) (xy 157.48 72.39)
+			(xy 223.52 111.76) (xy 223.52 115.57)
 		)
 		(stroke
@@
 	(wire
 		(pts
-			(xy 223.52 111.76) (xy 223.52 115.57)
+			(xy 223.52 139.7) (xy 223.52 143.51)
 		)
 		(stroke
@@
 	(wire
 		(pts
-			(xy 223.52 139.7) (xy 223.52 143.51)
+			(xy 95.25 48.26) (xy 69.85 48.26)
 		)
 		(stroke
@@
 	(wire
 		(pts
-			(xy 95.25 48.26) (xy 69.85 48.26)
+			(xy 152.4 97.79) (xy 157.48 97.79)
 		)
 		(stroke
@@
 	(wire
 		(pts
+			(xy 111.76 87.63) (xy 116.84 87.63)
+		)
+		(stroke
+			(width 0)
+			(type default)
+		)
+	)
+	(wire
+		(pts
 			(xy 152.4 67.31) (xy 157.48 67.31)
 		)
@@
 	(hierarchical_label "display_extmode"
 		(shape output)
-		(at 111.76 87.63 180)
+		(at 157.48 97.79 0)
 		(effects
 			(font
 				(size 1.27 1.27)
 			)
-			(justify right)
+			(justify left)
 		)
 	)
@@
 	(hierarchical_label "display_extcomin"
 		(shape output)
-		(at 111.76 85.09 180)
+		(at 111.76 87.63 180)
 		(effects
 			(font
@@
 	(hierarchical_label "diaply_cs"
 		(shape output)
-		(at 157.48 64.77 0)
+		(at 111.76 85.09 180)
 		(effects
 			(font
 				(size 1.27 1.27)
 			)
-			(justify left)
+			(justify right)
 		)
 	)
@@
 		(dnp no)
 		(fields_autoplaced yes)
-		(property "Reference" "U4"
+		(property "Reference" "U20"
 			(at 139.3033 143.51 0)
 			(show_name no)
@@
 			(project "weather_station"
 				(path "/934dbf27-5b13-4be9-992c-a6264d0a607d/2b524250-e61e-417a-a8f6-4d01fda9d4b0"
-					(reference "U4")
+					(reference "U20")
 					(unit 1)
 				)
@@
 		(dnp no)
 		(fields_autoplaced yes)
-		(property "Reference" "SW1"
+		(property "Reference" "SW20"
 			(at 246.38 120.65 0)
 			(show_name no)
@@
 			(project "weather_station"
 				(path "/934dbf27-5b13-4be9-992c-a6264d0a607d/2b524250-e61e-417a-a8f6-4d01fda9d4b0"
-					(reference "SW1")
+					(reference "SW20")
 					(unit 1)
 				)
@@
 		(dnp no)
 		(fields_autoplaced yes)
-		(property "Reference" "X1"
+		(property "Reference" "X20"
 			(at 56.515 33.02 0)
 			(show_name no)
@@
 			(project "weather_station"
 				(path "/934dbf27-5b13-4be9-992c-a6264d0a607d/2b524250-e61e-417a-a8f6-4d01fda9d4b0"
-					(reference "X1")
+					(reference "X20")
 					(unit 1)
 				)
@@
 		(in_pos_files yes)
 		(dnp no)
-		(property "Reference" "J6"
+		(property "Reference" "J20"
 			(at 242.062 36.576 0)
 			(hide yes)
@@
 			(project "weather_station"
 				(path "/934dbf27-5b13-4be9-992c-a6264d0a607d/2b524250-e61e-417a-a8f6-4d01fda9d4b0"
-					(reference "J6")
+					(reference "J20")
 					(unit 1)
 				)

Commit message: Updated schematic with power supply capacitors
Parts:
- R29: value 1k -> 0
Changed lines of the file:
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@@
 			)
 		)
-		(property "Value" "1k"
+		(property "Value" "0"
 			(at 233.68 124.46 90)
 			(show_name no)

Commit message: Changed capacitor value display
Parts:
- C28: value 0.1uF -> 100nF
Changed lines of the file:
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@@
 			)
 		)
-		(property "Value" "0.1uF"
+		(property "Value" "100nF"
 			(at 227.33 137.1599 0)
 			(show_name no)
