File: Hardware/weather_station.kicad_pcb (KiCad board)
At the start: 2 copper layers, 54.4 x 89 mm, 30 parts, among them J20 JTAG_connector, J30 Conn_01x10_Pin, J40 USB_C_Receptacle_USB2.0_16P, J41 Conn_01x04, J42 Conn_01x04, SW20 SW_Push, U10 AZ1117CH2-3.3, U20 STM32F103RGTx, U40 USBLC6-2SC6, X20 831066657

Commit message: Initial commit for the software
Parts:
- C28, C30, C31: value 0.1uF -> 100nF
Routing:
- net GND: vias 509 -> 503
